Commit message: Added support for depth camera simulation

File: mbot_description/xacro/mbot.xacro (robot description, xacro)
@@ -237,5 +237,5 @@
   <joint name="hokuyo_joint" type="fixed">
     <axis xyz="0 0 1" />
-    <origin xyz="0.15 0 -0.1" rpy="0 0 0"/>
+    <origin xyz="0.15 0 -0.15" rpy="0 0 0"/>
     <parent link="head"/>
     <child link="hokuyo_link"/>
@@ -246,5 +246,5 @@
       <pose>0 0 0 0 0 0</pose>
       <visualize>true</visualize>
-      <update_rate>40</update_rate>
+      <update_rate>20</update_rate>
       <ray>
         <scan>
@@ -299,5 +299,7 @@
   </link>
   <joint name="camera_joint" type="fixed">
-    <origin xyz="0 -0.14 0" rpy="0 0 -1.57"/>
+    <!-- <origin xyz="0 -0.14 0" rpy="0 0 -1.57"/> -->
+    <origin xyz="0.15 0.0 -0.05" rpy="0 0 0"/>
+    <axis xyz="0 0 1" />
     <parent link="head"/>
     <child link="camera_link"/>
@@ -305,7 +307,45 @@
   <!-- camera -->
   <gazebo reference="camera_link">
-    <sensor type="camera" name="camera1">
-      <update_rate>15.0</update_rate>
-      <camera name="head">
+    <sensor type="depth" name="depth_camera">
+      <update_rate>20</update_rate>
+      <camera>
+        <horizontal_fov>1.047198</horizontal_fov>
+        <image>
+          <width>640</width>
+          <height>480</height>
+          <format>R8G8B8</format>
+        </image>
+        <clip>
+          <near>0.05</near>
+          <far>3</far>
+        </clip>
+      </camera>
+      <plugin name="camera_plugin" filename="libgazebo_ros_openni_kinect.so">
+        <baseline>0.2</baseline>
+        <alwaysOn>true</alwaysOn>
+        <updateRate>0.0</updateRate>
+        <cameraName>/camera_ir</cameraName>
+        <imageTopicName>/camera/depth/image_raw</imageTopicName>
+        <cameraInfoTopicName>/camera/depth/info</cameraInfoTopicName>
+        <depthImageTopicName>/camera/depth/image_depth</depthImageTopicName>
+        <depthImageInfoTopicName>/camera/depth/info_depth</depthImageInfoTopicName>
+        <pointCloudTopicName>/camera/depth/points</pointCloudTopicName>
+        <frameName>camera_link</frameName>
+        <pointCloudCutoff>0.05</pointCloudCutoff>
+        <distortionK1>0</distortionK1>
+        <distortionK2>0</distortionK2>
+        <distortionK3>0</distortionK3>
+        <distortionT1>0</distortionT1>
+        <distortionT2>0</distortionT2>
+        <CxPrime>0</CxPrime>
+        <Cx>0</Cx>
+        <Cy>0</Cy>
+        <focalLength>0</focalLength>
+        <hackBaseline>0</hackBaseline>
+      </plugin>
+    </sensor>
+    <sensor type="camera" name="rgb_camera">
+      <update_rate>20.0</update_rate>
+      <camera>
         <horizontal_fov>1.3962634</horizontal_fov>
         <image>
@@ -320,7 +360,4 @@
         <noise>
           <type>gaussian</type>
-          <!-- Noise is sampled independently per pixel on each frame.
-               That pixel's noise value is added to each of its color
-               channels, which at that point lie in the range [0,1]. -->
           <mean>0.0</mean>
           <stddev>0.007</stddev>
@@ -330,7 +367,7 @@
         <alwaysOn>true</alwaysOn>
         <updateRate>0.0</updateRate>
-        <cameraName>mbot/camera1</cameraName>
-        <imageTopicName>image_raw</imageTopicName>
-        <cameraInfoTopicName>camera_info</cameraInfoTopicName>
+        <cameraName>/camera_rgb</cameraName>
+        <imageTopicName>/camera/rgb/image_raw</imageTopicName>
+        <cameraInfoTopicName>/camera/rgb/info</cameraInfoTopicName>
         <frameName>camera_link</frameName>
         <hackBaseline>0.07</hackBaseline>
